File: 555timer.sch (KiCad schematic (older format))
At the start: 10 parts, among them U1 NE555P

Commit message: Added all the traces, power planes and rearenged the silkscreen text
Parts:
- PWM1: value Conn_01x02_Female -> PWM
- R1: renamed from 1k1; value R1 -> 1k
Changed lines of the file:
@@
 $EndDescr
 $Comp
-L Device:R 1k1
+L Device:R R1
 U 1 1 61C1E5C1
 P 6550 3300
-F 0 "1k1" H 6480 3346 50  0000 R CNN
-F 1 "R1" H 6480 3255 50  0000 R CNN
+F 0 "R1" H 6480 3346 50  0000 R CNN
+F 1 "1k" H 6480 3255 50  0000 R CNN
 F 2 "Resistor_THT:R_Axial_DIN0207_L6.3mm_D2.5mm_P10.16mm_Horizontal" V 6480 3300 50  0001 C CNN
 F 3 "~" H 6550 3300 50  0001 C CNN
@@
 P 6550 3850
 F 0 "R_POT1" V 6343 3850 50  0000 C CNN
-F 1 "R_POT" V 6434 3850 50  0000 C CNN
+F 1 "R_POT" V 6434 3850 50  0001 C CNN
 F 2 "Potentiometer_THT:Potentiometer_Alps_RK163_Single_Horizontal" H 6550 3850 50  0001 C CNN
 F 3 "~" H 6550 3850 50  0001 C CNN
@@
 P 6300 3650
 F 0 "D1" V 6254 3570 50  0000 R CNN
-F 1 "D" V 6345 3570 50  0000 R CNN
+F 1 "D" V 6345 3570 50  0001 R CNN
 F 2 "Diode_THT:D_DO-15_P10.16mm_Horizontal" H 6300 3650 50  0001 C CNN
 F 3 "~" H 6300 3650 50  0001 C CNN
@@
 P 6800 3650
 F 0 "D2" V 6846 3730 50  0000 L CNN
-F 1 "D" V 6755 3730 50  0000 L CNN
+F 1 "D" V 6755 3730 50  0001 L CNN
 F 2 "Diode_THT:D_DO-15_P10.16mm_Horizontal" H 6800 3650 50  0001 C CNN
 F 3 "~" H 6800 3650 50  0001 C CNN
@@
 P 7750 3650
 F 0 "PWM1" H 7778 3626 50  0000 L CNN
-F 1 "Conn_01x02_Female" H 7778 3535 50  0000 L CNN
+F 1 "PWM" H 7778 3535 50  0001 L CNN
 F 2 "Connector_PinHeader_2.54mm:PinHeader_1x02_P2.54mm_Vertical" H 7750 3650 50  0001 C CNN
 F 3 "~" H 7750 3650 50  0001 C CNN
@@
 Connection ~ 2750 3500
 $Comp
-L power:GND #PWR?
+L power:GND #PWR0101
 U 1 1 61C5462C
 P 2750 3800
-F 0 "#PWR?" H 2750 3550 50  0001 C CNN
+F 0 "#PWR0101" H 2750 3550 50  0001 C CNN
 F 1 "GND" H 2755 3627 50  0000 C CNN
 F 2 "" H 2750 3800 50  0001 C CNN
@@
 Connection ~ 2750 3800
 $Comp
-L power:VDC #PWR?
+L power:VDC #PWR0104
 U 1 1 61C58BE7
 P 7300 3550
-F 0 "#PWR?" H 7300 3450 50  0001 C CNN
+F 0 "#PWR0104" H 7300 3450 50  0001 C CNN
 F 1 "VDC" H 7315 3723 50  0000 C CNN
 F 2 "" H 7300 3550 50  0001 C CNN
@@
 $EndComp
 $Comp
-L power:VDC #PWR?
+L power:VDC #PWR0105
 U 1 1 61C5862C
 P 5700 3200
-F 0 "#PWR?" H 5700 3100 50  0001 C CNN
+F 0 "#PWR0105" H 5700 3100 50  0001 C CNN
 F 1 "VDC" H 5715 3373 50  0000 C CNN
 F 2 "" H 5700 3200 50  0001 C CNN
@@
 	7550 3550 7300 3550
 $Comp
-L power:GND #PWR?
+L power:GND #PWR0106
 U 1 1 61C5B83F
 P 7300 3800
-F 0 "#PWR?" H 7300 3550 50  0001 C CNN
+F 0 "#PWR0106" H 7300 3550 50  0001 C CNN
 F 1 "GND" H 7305 3627 50  0000 C CNN
 F 2 "" H 7300 3800 50  0001 C CNN
@@
 	7550 3800 7300 3800
 $Comp
-L power:VCC #PWR?
+L power:VCC #PWR0107
 U 1 1 61C605C8
 P 2750 3400
-F 0 "#PWR?" H 2750 3250 50  0001 C CNN
+F 0 "#PWR0107" H 2750 3250 50  0001 C CNN
 F 1 "VCC" H 2765 3573 50  0000 C CNN
 F 2 "" H 2750 3400 50  0001 C CNN
@@
 $EndComp
 $Comp
-L power:VCC #PWR?
+L power:VCC #PWR0108
 U 1 1 61C61127
 P 5200 2850
-F 0 "#PWR?" H 5200 2700 50  0001 C CNN
+F 0 "#PWR0108" H 5200 2700 50  0001 C CNN
 F 1 "VCC" H 5215 3023 50  0000 C CNN
 F 2 "" H 5200 2850 50  0001 C CNN
@@
 $EndComp
 $Comp
-L power:VCC #PWR?
+L power:VCC #PWR0109
 U 1 1 61C62022
 P 6550 3050
-F 0 "#PWR?" H 6550 2900 50  0001 C CNN
+F 0 "#PWR0109" H 6550 2900 50  0001 C CNN
 F 1 "VCC" H 6565 3223 50  0000 C CNN
 F 2 "" H 6550 3050 50  0001 C CNN
@@
 $EndComp
 $Comp
-L power:VCC #PWR?
+L power:VCC #PWR0110
 U 1 1 61C62C93
 P 4600 3650
-F 0 "#PWR?" H 4600 3500 50  0001 C CNN
+F 0 "#PWR0110" H 4600 3500 50  0001 C CNN
 F 1 "VCC" H 4615 3823 50  0000 C CNN
 F 2 "" H 4600 3650 50  0001 C CNN
